Commit message: Docuementación archivos en ingles

File: dsr_description/xacro/macro.m1013.white.xacro (robot description, xacro)
@@ -40,10 +40,4 @@
 				<inertia ixx="0.039" ixy="2.1e-05" ixz="-3.61e-05" iyy="0.023" iyz="-0.003" izz="0.039" />
 			</inertial>
-			<collision>
-				<origin rpy="0 0 0" xyz="0 0 0" />
-				<geometry>
-					<mesh filename="package://dsr_description/meshes/m1013_white/MF1013_1_0.stl" scale="0.001 0.001 0.001" />
-				</geometry>
-			</collision>
 			<visual>
 				<origin rpy="0 0 0" xyz="0 0 0" />
@@ -68,22 +62,4 @@
 				<inertia ixx="0.820" ixy="1.19e-05" ixz="-0.000263" iyy="0.82" iyz="-0.008" izz="0.031" />
 			</inertial>
-			<collision>
-				<origin rpy="0 0 0" xyz="0 0 0" />
-				<geometry>
-					<mesh filename="package://dsr_description/meshes/m1013_white/MF1013_2_0.stl" scale="0.001 0.001 0.001" />
-				</geometry>
-			</collision>
-			<collision>
-				<origin rpy="0 0 0" xyz="0 0 0" />
-				<geometry>
-					<mesh filename="package://dsr_description/meshes/m1013_white/MF1013_2_1.stl" scale="0.001 0.001 0.001" />
-				</geometry>
-			</collision>
-			<collision>
-				<origin rpy="0 0 0" xyz="0 0 0" />
-				<geometry>
-					<mesh filename="package://dsr_description/meshes/m1013_white/MF1013_2_2.stl" scale="0.001 0.001 0.001" />
-				</geometry>
-			</collision>
 			<visual>
 				<origin rpy="0 0 0" xyz="0 0 0" />
@@ -120,10 +96,4 @@
 				<inertia ixx="0.012" ixy="-4.38e-06" ixz="-1.2e-06" iyy="0.008" iyz="0.002" izz="0.011" />
 			</inertial>
-			<collision>
-				<origin rpy="0 0 0" xyz="0 0 0" />
-				<geometry>
-					<mesh filename="package://dsr_description/meshes/m1013_white/MF1013_3_0.stl" scale="0.001 0.001 0.001" />
-				</geometry>
-			</collision>
 			<visual>
 				<origin rpy="0 0 0" xyz="0 0 0" />
@@ -148,16 +118,4 @@
 				<inertia ixx="0.177" ixy="-2.34e-06" ixz="-4.92e-06" iyy="0.161" iyz="-0.05" izz="0.022" />
 			</inertial>
-			<collision>
-				<origin rpy="0 0 0" xyz="0 0 0" />
-				<geometry>
-					<mesh filename="package://dsr_description/meshes/m1013_white/MF1013_4_0.stl" scale="0.001 0.001 0.001" />
-				</geometry>
-			</collision>
-			<collision>
-				<origin rpy="0 0 0" xyz="0 0 0" />
-				<geometry>
-					<mesh filename="package://dsr_description/meshes/m1013_white/MF1013_4_1.stl" scale="0.001 0.001 0.001" />
-				</geometry>
-			</collision>
 			<visual>
 				<origin rpy="0 0 0" xyz="0 0 0" />
@@ -188,10 +146,4 @@
 				<inertia ixx="0.007" ixy="-4.93e-06" ixz="-5.57e-06" iyy="0.004" iyz="-6.64e-05" izz="0.007" />
 			</inertial>
-			<collision>
-				<origin rpy="0 0 0" xyz="0 0 0" />
-				<geometry>
-					<mesh filename="package://dsr_description/meshes/m1013_white/MF1013_5_0.stl" scale="0.001 0.001 0.001" />
-				</geometry>
-			</collision>
 			<visual>
 				<origin rpy="0 0 0" xyz="0 0 0" />
@@ -216,10 +168,4 @@
 				<inertia ixx="0.001" ixy="-2.79e-06" ixz="5.78e-06" iyy="0.001" iyz="-6.67e-06" izz="0.001" />
 			</inertial>
-			<collision>
-				<origin rpy="0 0 0" xyz="0 0 0" />
-				<geometry>
-					<mesh filename="package://dsr_description/meshes/m1013_white/MF1013_6_0.stl" scale="0.001 0.001 0.001" />
-				</geometry>
-			</collision>
 			<visual>
 				<origin rpy="0 0 0" xyz="0 0 0" />
